Commit message: "Feat: fix bug"

File: rsc/raibo2/urdf/raibo2.urdf (robot description, URDF)
Before this commit: robot raibo2, 17 links, 16 joints
Links:
- link LF_SHANK: geometry collision box size=0.07 0.02586 0.029; collision box size=0.2965 0.02586 0.029
- link LH_SHANK: geometry collision box size=0.07 0.02586 0.029; collision box size=0.2965 0.02586 0.029
- link RF_SHANK: geometry collision box size=0.07 0.02586 0.029; collision box size=0.2965 0.02586 0.029
- link RH_SHANK: geometry collision box size=0.07 0.02586 0.029; collision box size=0.2965 0.02586 0.029
Joints:
- joint LF_HFE: limit lower=-6.2832 upper=6.2832 effort=90.8558 velocity=31.5 -> lower=-2.428 upper=3.185 effort=90.8558 velocity=31.5
- joint LH_HFE: limit lower=-6.2832 upper=6.2832 effort=90.8558 velocity=31.5 -> lower=-1.639 upper=3.972 effort=90.8558 velocity=31.5
- joint RF_HFE: limit lower=-6.2832 upper=6.2832 effort=90.8558 velocity=31.5 -> lower=-2.428 upper=3.185 effort=90.8558 velocity=31.5
- joint RH_HFE: limit lower=-6.2832 upper=6.2832 effort=90.8558 velocity=31.5 -> lower=-1.639 upper=3.972 effort=90.8558 velocity=31.5
